Commit message: chore: include autogenerated URDF and scene files in commit

File: dual_arm_moveit_config/config/dual_arm_world.urdf (robot description, URDF)
Before this commit: robot dual_arm_disassembly_cell, 36 links, 35 joints
Links:
- link ft_ft300_mounting_plate: geometry collision mesh filename=file:///home/adip/workspace/dev_ws/install/robotiq_ft_senso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; visual mesh filename=file:///home/adip/workspace/dev_ws/install/robotiq_ft_senso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
- link ft_ft300_sensor: geometry collision mesh filename=file:///home/adip/workspace/dev_ws/install/robotiq_ft_senso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; visual mesh filename=file:///home/adip/workspace/dev_ws/install/robotiq_ft_senso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

File: scene_description/urdf/scene.urdf (robot description, URDF)
Before this commit: robot scene, 2 links, 1 joints
Links:
- link base_link: geometry collision mesh filename=file:///home/adip/workspace/dev_ws/src/scene_description/me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 scale=0.001 0.001 0.001; visual mesh filename=file:///home/adip/workspace/dev_ws/src/scene_description/me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 scale=0.001 0.001 0.001
